File: keyboard/monarch/doc/Monarch.brd (EAGLE design)
At the start: 359 x 95.3 mm, 186 parts, among them J1 MINIUSB, U2 ATMEGA32U4, Y1 16MHZ

Commit message: Update the Monarch docs to revision 10 of the board
Parts:
- added +5V: (no value), Seeed-OPL-Connector:H2-2.54
- moved C6 5.41 mm to (62.8, -36.5), turned to 270 degrees
Connections:
- net GND: now also +5V.1
- net VCC: now also +5V.2
Routing:
- net VCC: track 70.3 -> 116.1 mm, vias 6 -> 8
- net GND: track 94.4 -> 83.9 mm, vias 1 -> 0
Other:
- board text added: "GND"
- board text added: "VCC"
Changed lines of the file:
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@@
 <rectangle x1="201.3966" y1="-90.551" x2="202.1078" y2="-90.5002" layer="22" rot="R180"/>
 <rectangle x1="198.9074" y1="-90.551" x2="199.6186" y2="-90.5002" layer="22" rot="R180"/>
-<text x="12.25" y="-68" size="2.1844" layer="21" font="vector">Designed by skullY in Felton, CA</text>
+<text x="29.25" y="-29.5" size="2.1844" layer="21" font="vector">Designed by skullY in Felton, CA</text>
+<text x="66.1" y="-77.5" size="1.778" layer="21" rot="R270">GND</text>
+<text x="66.1" y="-67.4" size="1.778" layer="21" rot="R270">VCC</text>
 </plain>
 <attributes>
@@
 <attribute name="MPN" value="CC0805KRX7R9BB104" x="32.5" y="-75.75" size="1.778" layer="28" rot="MR180" display="off"/>
 </element>
-<element name="C6" library="Seeed-OPL-Capacitor" package="C0805" value="100nf" x="61" y="-31.35" rot="MR90">
-<attribute name="MPN" value="CC0805KRX7R9BB104" x="103" y="-75.35" size="1.778" layer="28" rot="MR90" display="off"/>
+<element name="C6" library="Seeed-OPL-Capacitor" package="C0805" value="100nf" x="62.8" y="-36.45" rot="MR270">
+<attribute name="MPN" value="CC0805KRX7R9BB104" x="20.8" y="7.55" size="1.778" layer="28" rot="MR270" display="off"/>
 </element>
 <element name="C7" library="Seeed-OPL-Capacitor" package="C0805" value="100nf" x="75.3" y="-24.25" rot="MR0">
@@
 <element name="C1" library="Seeed-OPL-Capacitor" package="C0805" value="1uf" x="62.8" y="-18.5" rot="MR0">
 <attribute name="MPN" value="CC0805KKX7R8BB105" x="62.8" y="-18.5" size="1.778" layer="28" rot="MR0" display="off"/>
+</element>
+<element name="+5V" library="Seeed-OPL-Connector" package="H2-2.54" value="" x="67" y="-75" rot="R180">
+<attribute name="MPN" value="F185-1102A1BSYA1" x="67" y="-75" size="1.778" layer="27" rot="R180" display="off"/>
 </element>
 </elements>
@@
 <wire x1="64" y1="-102.901" x2="59.3" y2="-102.901" width="0.3" layer="16"/>
 <wire x1="65.4" y1="-31.6" x2="65.4" y2="-37.6" width="0.3" layer="16"/>
-<wire x1="65.4" y1="-37.6" x2="64.25" y2="-38.75" width="0.3" layer="16"/>
 <via x="64.25" y="-38.75" extent="1-16" drill="0.6"/>
 <wire x1="64.25" y1="-38.75" x2="64.25" y2="-102.651" width="0.3" layer="1"/>
 <wire x1="64.25" y1="-102.651" x2="64" y2="-102.901" width="0.3" layer="1"/>
 <via x="64" y="-102.901" extent="1-16" drill="0.6"/>
+<wire x1="65.4" y1="-37.6" x2="64.25" y2="-38.75" width="0.3" layer="16"/>
+<wire x1="64.25" y1="-38.75" x2="64.2" y2="-38.8" width="0.3" layer="16"/>
+<wire x1="64.2" y1="-38.8" x2="64.2" y2="-38.7" width="0.3" layer="16"/>
+<wire x1="64.2" y1="-38.7" x2="64.25" y2="-38.75" width="0.3" layer="16"/>
 </signal>
 <signal name="N$70">
@@
 <wire x1="62.75" y1="-10.75" x2="62.69" y2="-10.69" width="0.3" layer="16"/>
 <wire x1="62.69" y1="-10.69" x2="62.69" y2="-10.666" width="0.3" layer="16"/>
-<wire x1="64.05" y1="-30.25" x2="61.111" y2="-30.25" width="0.3" layer="16"/>
-<wire x1="61.111" y1="-30.25" x2="60.111" y2="-31.35" width="0.3" layer="16"/>
 <wire x1="63.5" y1="-34.639" x2="63.4" y2="-34.639" width="0.3" layer="16"/>
-<wire x1="63.4" y1="-34.639" x2="60.111" y2="-31.35" width="0.3" layer="16"/>
 <wire x1="70.75" y1="-27.25" x2="68.5" y2="-27.25" width="0.3" layer="16"/>
 <wire x1="68.0748" y1="-15.619" x2="68.0748" y2="-17" width="0.3" layer="16"/>
@@
 <wire x1="80.25" y1="-22.25" x2="80.25" y2="-22.639" width="0.3" layer="16"/>
 <wire x1="80.25" y1="-22.639" x2="80.611" y2="-23" width="0.3" layer="16"/>
-<via x="58.75" y="-31.5" extent="1-16" drill="0.6"/>
-<wire x1="60.111" y1="-31.35" x2="58.9" y2="-31.35" width="0.3" layer="16"/>
-<wire x1="58.9" y1="-31.35" x2="58.75" y2="-31.5" width="0.3" layer="16"/>
 <wire x1="64.05" y1="-26.25" x2="62.75" y2="-26.25" width="0.3" layer="16"/>
 <wire x1="62.75" y1="-26.25" x2="61.5" y2="-25" width="0.3" layer="16"/>
@@
 </polygon>
 <contactref element="C1" pad="2"/>
+<contactref element="+5V" pad="1"/>
 </signal>
 <signal name="N$77">
@@
 <wire x1="70.5" y1="-34.639" x2="70.639" y2="-34.639" width="0.3" layer="16"/>
 <wire x1="70.639" y1="-34.639" x2="72" y2="-36" width="0.3" layer="16"/>
-<wire x1="64.05" y1="-30.75" x2="62.489" y2="-30.75" width="0.3" layer="16"/>
-<wire x1="62.489" y1="-30.75" x2="61.889" y2="-31.35" width="0.3" layer="16"/>
 <via x="63.3" y="-31.4" extent="1-16" drill="0.6"/>
 <wire x1="63.3" y1="-31.4" x2="63.3" y2="-24.8" width="0.3" layer="1"/>
@@
 <wire x1="64.05" y1="-30.75" x2="63.95" y2="-30.75" width="0.3" layer="16"/>
 <wire x1="63.95" y1="-30.75" x2="63.3" y2="-31.4" width="0.3" layer="16"/>
+<wire x1="63.3" y1="-31.4" x2="62.8" y2="-31.4" width="0.3" layer="16"/>
+<wire x1="62.8" y1="-31.4" x2="61.9" y2="-32.3" width="0.3" layer="16"/>
+<wire x1="61.9" y1="-32.3" x2="61.9" y2="-36.439" width="0.3" layer="16"/>
+<wire x1="61.9" y1="-36.439" x2="61.911" y2="-36.45" width="0.3" layer="16"/>
+<contactref element="+5V" pad="2"/>
+<wire x1="61.911" y1="-36.45" x2="62" y2="-36.539" width="0.3" layer="16"/>
+<wire x1="62" y1="-36.539" x2="62" y2="-38.7" width="0.3" layer="16"/>
+<via x="62" y="-38.7" extent="1-16" drill="0.6" shape="square"/>
+<wire x1="62" y1="-38.7" x2="62" y2="-73.7" width="0.3" layer="1"/>
+<via x="62" y="-73.7" extent="1-16" drill="0.6"/>
+<wire x1="62" y1="-73.7" x2="62.03" y2="-73.73" width="0.3" layer="16"/>
+<wire x1="62.03" y1="-73.73" x2="67" y2="-73.73" width="0.3" layer="16"/>
 </signal>
 </signals>

Commit message: Updating the monarch design files
Parts:
- removed +5V: (no value), Seeed-OPL-Connector:H2-2.54
- added FET5: MOSFET, smd-ipc:SOT23
- added J2: 3p-2.54, Seeed-OPL-Connector:H3-2.54
- added J3: (no value), Seeed-OPL-Connector:H2-2.54
- added J4: 5p-2.54, Seeed-OPL-Connector:H4-2.54
- added LED1, LED10, LED11, LED12, LED13, LED14, LED15, LED16, LED2, LED3, LED4, LED5, LED6, LED7, LED8, LED9: (no value), AlpsCherry:P-SMD-LED-GENERIC
- added R10, R11, R12, R13, R14, R15, R16, R17, R18, R19, R5, R6, R7, R8, R9: 100R, Seeed-OPL-Resistor:R0805
- added R20: 10K, Seeed-OPL-Resistor:R0805
- added R4: (no value), Seeed-OPL-Resistor:R0805
- moved RLCAPSLOCK 11.6 mm to (91.4, -70.2)
- moved RLCLEAR 11.5 mm to (91.4, -73.5)
- moved DSPACE_6.25 7.00 mm to (226.3, -101.2)
Connections:
- new net LED1: J4.3, U2.30
- new net LED2: J4.2, U2.31
- new net N$100: LED11.MINUS, R14.2
- new net N$101: LED10.MINUS, R13.2
- new net N$102: LED9.MINUS, R12.2
- new net N$103: LED8.MINUS, R11.2
- new net N$104: LED7.MINUS, R10.2
- new net N$105: LED14.MINUS, R17.2
- new net N$106: LED13.MINUS, R16.2
- new net N$154: FET5.1, J2.1, J3.1, R20.2
- new net N$91: LED1.MINUS, R4.2
- new net N$92: LED2.MINUS, R5.2
- new net N$93: LED3.MINUS, R6.2
- new net N$94: LED4.MINUS, R7.2
- new net N$95: LED5.MINUS, R8.2
- new net N$96: LED6.MINUS, R9.2
- new net N$97: LED15.MINUS, R18.2
- new net N$98: LED16.MINUS, R19.2
- new net N$99: LED12.MINUS, R15.2
- new net UNDERLIGHT: FET5.3, J3.2, R10.1, R11.1, R12.1, R13.1, R14.1, R15.1, R16.1, R17.1, R18.1, R19.1, R4.1, R5.1, R6.1, R7.1, R8.1, R9.1
- net GND: now also FET5.2, J4.1, R20.1; no longer +5V.1
- net N$86: now also J2.2; no longer U2.30
- net N$90: now also J2.3; no longer U2.31
- net VCC: now also J4.4, LED1.PLUS, LED10.PLUS, LED11.PLUS, LED12.PLUS, LED13.PLUS, LED14.PLUS, LED15.PLUS, LED16.PLUS, LED2.PLUS, LED3.PLUS, LED4.PLUS, LED5.PLUS, LED6.PLUS, LED7.PLUS, LED8.PLUS, LED9.PLUS; no longer +5V.2
Routing:
- net VCC: track 116.1 -> 1091.0 mm, vias 8 -> 26
- net UNDERLIGHT: track 0.00 -> 874.1 mm
- net LED2: track 0.00 -> 56.3 mm, vias 0 -> 2
- net LED1: track 0.00 -> 52.8 mm, vias 0 -> 2
- net N$90: track 44.1 -> 2.55 mm, vias 1 -> 0
- net N$86: track 39.9 -> 2.40 mm, vias 1 -> 0
- net N$154: track 0.00 -> 36.3 mm, vias 0 -> 1
- net GND: track 83.9 -> 64.3 mm, vias 0 -> 1
- net LCLEAR: track 103.6 -> 116.8 mm
- net LCAPSLOCK: track 16.7 -> 6.98 mm
- net N$102: track 0.00 -> 8.81 mm
- net N$99: track 0.00 -> 4.17 mm
- net N$101: track 0.00 -> 4.17 mm
- net N$100: track 0.00 -> 4.17 mm
- net N$105: track 0.00 -> 4.17 mm
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Other:
- board text added: "B6"
- board text added: "C6"
- board text added: "RLCAPSLOCK"
- board text added: "RLCLEAR"
- board text added: "UNDERLIGHT"

Commit message: Update the monarch schematic and layout
Parts:
- removed J1: MINIUSB, Seeed-OPL-Connector:MINIUSB5+4P-0.8-90D
- added X1: MINI-USB-UX60-MB-5S8, con-hirose:UX60-MB-5S8
- moved C6 3.00 mm to (62.8, -39.5)
- moved R3 2.00 mm to (63.5, -35.8)
- moved C5 1.00 mm to (70.5, -34.8)
- moved RLCAPSLOCK 0.28 mm to (91.6, -70.4)
- moved RLCLEAR 0.28 mm to (91.6, -73.7)
- renumbered FET5 to FET1, RCMD1 to RCMD, U2 to U1
Connections:
- net GND: now also X1.5; no longer J1.5, J1.GND@1, J1.GND@2, J1.GND@3, J1.GND@4
- net N$88: now also X1.3; no longer J1.3
- net N$89: now also X1.2; no longer J1.2
- net VCC: now also X1.1; no longer J1.1
Routing:
- net GND: track 64.3 -> 54.9 mm, vias 1 -> 2
- net UNDERLIGHT: track 874.1 -> 867.8 mm
- net VCC: track 1091.0 -> 1092.5 mm
- net N$83: track 2.33 -> 3.84 mm
- net COLUMN17: track 402.9 -> 401.4 mm
- net LCAPSLOCK: track 6.98 -> 6.06 mm
- net N$89: track 2.20 -> 2.89 mm
- net LCLEAR: track 116.8 -> 117.4 mm
Other:
- board text added: "FET Bypass Jumper these pins if UNDERLIGHT is connected to VCC."
- board text added: "LALT"
- board text added: "LCMD"
- board text added: "RALT"
